File: food_dispenser.sch (EAGLE design)
At the start: 25 parts, among them IC1 PCF8574T, M1 SERVO

Commit message: remove redundant sheet
Parts:
- removed NODE1: NODEMCU_ESP8266, nodemcu_esp8266:NODEMCU_ESP8266
Connections:
- net +3V3: no longer NODE1.3V3@1
Changed lines of the file:
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@@
 </classes>
 <parts>
-<part name="NODE1" library="nodemcu_esp8266" deviceset="NODEMCU_ESP8266" device=""/>
-<part name="P+1" library="supply1" library_urn="urn:adsk.eagle:library:371" deviceset="+5V" device=""/>
-<part name="+3V1" library="supply1" library_urn="urn:adsk.eagle:library:371" deviceset="+3V3" device=""/>
 <part name="IC1" library="micro-philips" deviceset="PCF8574" device="T"/>
 <part name="R2" library="adafruit" deviceset="R-US_" device="R0805" value="100"/>
@@
 <sheet>
 <plain>
-</plain>
-<instances>
-<instance part="NODE1" gate="G$1" x="63.5" y="60.96" smashed="yes">
-<attribute name="VALUE" x="53.34" y="33.02" size="1.27" layer="96"/>
-<attribute name="NAME" x="53.34" y="78.74" size="1.27" layer="95"/>
-</instance>
-<instance part="P+1" gate="1" x="88.9" y="83.82" smashed="yes">
-<attribute name="VALUE" x="86.36" y="78.74" size="1.778" layer="96" rot="R90"/>
-</instance>
-<instance part="+3V1" gate="G$1" x="35.56" y="81.28" smashed="yes">
-<attribute name="VALUE" x="33.02" y="76.2" size="1.778" layer="96" rot="R90"/>
-</instance>
-</instances>
-<busses>
-</busses>
-<nets>
-<net name="+3V3" class="0">
-<segment>
-<pinref part="+3V1" gate="G$1" pin="+3V3"/>
-<pinref part="NODE1" gate="G$1" pin="3V3@1"/>
-<wire x1="35.56" y1="78.74" x2="35.56" y2="73.66" width="0.1524" layer="91"/>
-<wire x1="35.56" y1="73.66" x2="48.26" y2="73.66" width="0.1524" layer="91"/>
-</segment>
-</net>
-</nets>
-</sheet>
-<sheet>
-<plain>
